File: electronics/KiCad/1_Distribution_Board/1_Distribution_Board.kicad_pcb (KiCad board)
At the start: 2 copper layers, 130 x 120 mm, 193 parts, among them CN1 HC-5264-3A, CN2 HC-5264-3A, J1 JST VH, J10 Generic 2.54mm, J11 Generic 2.54mm, J12 Conn_01x06, J13 Conn_01x10, J14 2.54-1*4P母, J15 2.54-1*4P母, J16 PM254V-11-06-H85, J17 Conn_02x08_Odd_Even, J18 PM254V-11-06-H85, J19 2.54-1*4P母, J2 JST VH, J20 2.54-1*4P母, J21 Jumper Pins, J22 Jumper Pins, J23 JST PH, J24 Generic 2.54mm, J25 Jumper Pins, J26 Jumper Pins, J27 JST PH, J28 Generic 2.54mm, J29 Jumper Pins, J3 JST VH, J30 Jumper Pins, J31 JST PH, J32 Generic 2.54mm, J33 Jumper Pins, J34 Jumper Pins, J35 JST PH, J36 Generic 2.54mm, J37 Jumper Pins, J38 Jumper Pins, J39 JST PH, J4 Conn_01x04, J40 Generic 2.54mm, J5 Generic 2.54mm, J6 Generic 2.54mm, J8 Generic 2.54mm, J9 Generic 2.54mm, M1 MountingHole_3.2mm_M3_ISO7380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, P1 Header-Female-2.54_1x8, P10 Header-Female-2.54_1x8, P11 Header-Female-2.54_1x2, P12 Header-Female-2.54_1x8, P13 Header-Female-2.54_1x8, P14 Header-Female-2.54_1x2, P15 Header-Female-2.54_1x8, P2 Header-Female-2.54_1x2, P3 Header-Female-2.54_1x8, P4 Header-Female-2.54_1x8, P5 Header-Female-2.54_1x2, P6 Header-Female-2.54_1x8, P7 Header-Female-2.54_1x8, P8 Header-Female-2.54_1x2, P9 Header-Female-2.54_1x8, Q1 DMG2305UX, Q2 AO3400A, Q3 AO3400A, Q4 AO3400A, Q5 AO3400A, U1 KH-2.54FH-1X20P-H8.5, U2 KH-2.54FH-1X20P-H8.5, U3 R-78C5.0-1.0, U4 R-78B12-2.0, U5 R-78B6.5-1.5, U6 PCA9306, U7 PCA9685PW, Y1 25MHz

Commit message: Distribution board v1.4.1: effreek's revision, REV label, JLC rotation offsets restored (#1169)
effreek's pull-up/pull-down cleanup and test serial-servo circuit (J11/J14/J15), REV 1.4.1 on the board, the 33 JLC rotation offsets restored, test points out of the position file, and the V1.4.1 Gerber zip. Supersedes #1042.

Co-authored-by: effreek <115494910+effreek@users.noreply.github.com>
Co-Authored-By: Claude Opus 5.5 <noreply@anthropic.com>
Parts:
- removed C8: 100nF, PCM_JLCPCB:C_0603
- removed J16, J18: PM254V-11-06-H85, EasyEDA:HDR-TH_6P-P2.54-V-F
- removed J19, J20: 2.54-1*4P母, EasyEDA:HDR-TH_4P-P2.54-V-F
- removed J21, J22, J25, J26, J29, J30, J33, J34, J37, J38: Jumper Pins, Connector_PinHeader_2.54mm:PinHeader_1x03_P2.54mm_Vertical
- removed J6: Generic 2.54mm, Connector_PinHeader_2.54mm:PinHeader_1x03_P2.54mm_Vertical
- removed JP1, JP2, JP3, JP4: ~, PCM_SparkFun-Jumper:Jumper_2_NO
- removed Q5: AO3400A, PCM_JLCPCB:Q_SOT-23
- removed R15: 100Ω, PCM_JLCPCB:R_0603
- removed R23: 1kΩ, PCM_JLCPCB:R_0603
- removed R26, R37, R39, R41, R59, R69, R70, R73, R74, R75, R76, R79, R80, R81, R82, R85, R86, R87, R88: 10kΩ, PCM_JLCPCB:R_0603
- J11: value Generic 2.54mm -> JST B02B-XASK; footprint Connector_PinHeader_2.54mm:PinHeader_1x02_P2.54mm_Vertical -> Connector_JST:JST_XA_B02B-XASK-1-A_1x02_P2.50mm_Vertical
- J14, J15: value 2.54-1*4P母 -> JST B02B-XASK; footprint EasyEDA:HDR-TH_4P-P2.54-V-F -> Connector_JST:JST_XA_B02B-XASK-1-A_1x02_P2.50mm_Vertical
- J5: value Generic 2.54mm -> 01x02 Dupont Latching; footprint Connector_PinHeader_2.54mm:PinHeader_1x03_P2.54mm_Vertical -> Connector_Molex:Molex_SL_171971-0002_1x02_P2.54mm_Vertical
- R12: value 10kΩ -> 0Ω
- R21, R22, R27, R28: value 180Ω -> 10kΩ; footprint PCM_JLCPCB:R_1206 -> PCM_JLCPCB:R_0603
- R33: value 10kΩ -> 2.2kΩ
- R35: value 10kΩ -> 100Ω
- moved R12 125.2 mm to (113.9, 140.5)
- moved R22 85.1 mm to (119.8, 41.2), turned to 0 degrees
- moved R21 84.0 mm to (119.8, 38.6), turned to 0 degrees
- moved R35 71.8 mm to (72.8, 36.0), turned to 90 degrees
- moved R64 71.2 mm to (119.8, 114.6)
- moved J15 70.7 mm to (41.6, 44.5), turned to 90 degrees
- moved R63 69.0 mm to (119.8, 112.1)
- moved R27 64.9 mm to (119.8, 63.1), turned to 0 degrees
- moved R28 63.3 mm to (119.8, 65.6), turned to 0 degrees
- moved J14 59.1 mm to (41.6, 55.6), turned to 90 degrees
- moved R68 58.6 mm to (60.4, 78.3), turned to 180 degrees
- moved R67 54.9 mm to (60.4, 80.8), turned to 180 degrees
- moved R33 50.4 mm to (80.7, 78.6), turned to 0 degrees
- moved R62 49.2 mm to (119.8, 90.1)
- moved R61 47.1 mm to (119.8, 87.5)
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Connections:
- net /GPIO3-GPIO_IN_HALL-SW_0 renamed /GPIO3-GPIO_IN-LIMIT_SWITCH
- C9 pad 2: +3V3 -> VSYS
- CN1 pad 1: /Power/WAVESHARE_DATA -> Net-(CN1-Pad1)
- CN2 pad 1: /Power/WAVESHARE_DATA -> /SERIAL_SERVO
- J10 pad 1: Net-(J10-Pin_1) -> +24V
- J11 pad 1: Net-(J11-Pin_1) -> +24V
- J14 pad 1: /PCA9685 Module/PWM_0 -> +24V
- J14 pad 2: /PCA9685 Module/PWM_1 -> Net-(J10-Pin_2)
- J15 pad 1: /PCA9685 Module/PWM_4 -> +24V
- J15 pad 2: /PCA9685 Module/PWM_5 -> Net-(J15-Pin_2)
- J8 pad 1: Net-(J8-Pin_1) -> +24V
- J8 pad 2: Net-(J8-Pin_2) -> Net-(J11-Pin_2)
- J9 pad 1: Net-(J9-Pin_1) -> +24V
- J9 pad 2: Net-(J9-Pin_2) -> Net-(J15-Pin_2)
- Q2 pad 3: Net-(J8-Pin_2) -> Net-(J11-Pin_2)
- Q3 pad 3: Net-(J9-Pin_2) -> Net-(J15-Pin_2)
- R12 pad 1: +3V3 -> Net-(CN1-Pad1)
- R12 pad 2: Net-(J6-Pin_2) -> /SERIAL_SERVO
- R21 pad 1: +24V -> GND
- R21 pad 2: Net-(J8-Pin_1) -> /Stepper Module/MS1
- R22 pad 1: +24V -> GND
- R22 pad 2: Net-(J9-Pin_1) -> /Stepper Module/MS2
- R27 pad 1: +24V -> +3V3
- R27 pad 2: Net-(J10-Pin_1) -> /Stepper Module1/MS1
- R28 pad 1: +24V -> GND
- R28 pad 2: Net-(J11-Pin_1) -> /Stepper Module1/MS2
- R33 pad 1: VSYS -> /SERIAL_SERVO
- R33 pad 2: /PCA9685 Module/A0 -> +3V3
- R35 pad 1: VSYS -> /SERIAL_SERVO
- R35 pad 2: /PCA9685 Module/A1 -> /GPIO2-GPIO_IN_OUT-SERIAL_SERVO
- R61 pad 1: +3V3 -> GND
- R61 pad 2: Net-(J21-Pin_1) -> /Stepper Module2/MS1
- R62 pad 1: Net-(J21-Pin_3) -> +3V3
- R62 pad 2: GND -> /Stepper Module2/MS2
- R63 pad 2: Net-(J22-Pin_1) -> /Stepper Module3/MS1
- R64 pad 1: Net-(J22-Pin_3) -> +3V3
- R64 pad 2: GND -> /Stepper Module3/MS2
- R67 pad 1: +3V3 -> GND
- R67 pad 2: Net-(J25-Pin_1) -> /Stepper Module4/MS1
- R68 pad 1: Net-(J25-Pin_3) -> GND
- R68 pad 2: GND -> /Stepper Module4/MS2
- U1 pad 4: /GPIO2-GPIO_IN_HALL-SW_1 -> /GPIO2-GPIO_IN_OUT-SERIAL_SERVO
- Y1 pad 1: +3V3 -> VSYS
- Y1 pad 4: +3V3 -> VSYS
Routing:
- net /SERIAL_SERVO: track 0.00 -> 163.4 mm, vias 0 -> 4
- net +3V3: track 478.5 -> 383.7 mm, vias 19 -> 18
- net VSYS: track 170.5 -> 120.4 mm
- net /PCA9685 Module/~{OE}: track 43.4 -> 7.36 mm
- net /GPIO3-GPIO_IN-LIMIT_SWITCH: track 43.3 -> 9.12 mm
- net /GPIO1-GPIO_OUT-LED_0: track 60.8 -> 29.0 mm
- net /GPIO2-GPIO_IN_HALL-SW_1: track 27.3 -> 0.00 mm
- net /Power/WAVESHARE_DATA: track 24.7 -> 0.00 mm
- net /PCA9685 Module/I2C0_SCL_5V: track 42.1 -> 18.5 mm, vias 2 -> 0
- net /PCA9685 Module/I2C0_SDA_5V: track 38.2 -> 16.7 mm
- net GND: track 109.3 -> 89.8 mm, vias 56 -> 35
- net /PCA9685 Module/A0: track 30.6 -> 13.0 mm
- net /PCA9685 Module/A1: track 29.2 -> 12.6 mm
- net +24V: track 451.8 -> 437.7 mm, vias 5 -> 1
- net /PCA9685 Module/PWM_1: track 38.6 -> 25.4 mm
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Other:
- board text added: "1_Distribution_Board PCB REV 1.4.1"
- board text added: "1_Distribution_Board REV 1.4.1"
- board text added: "I2C Address (All pins Low)"
- board text added: "LIMIT SWITCH"
- board text added: "USB"
- board text added: "follow on instagram @basicallyhandle"
- board text removed: "!Double check!"
- board text removed: "1 2 3"
- board text removed: "1-2"
- board text removed: "1_Distribution_Board Assembly REV"
- board text removed: "1_Distribution_Board PCB REV 1.3"
- board text removed: "2-3"
- board text removed: "3 2 1"
- board text removed: "3.3V"
- board text removed: "3V3"
- board text removed: "A10"
- board text removed: "Bypass R21"
- board text removed: "Bypass R22"
- board text removed: "Bypass R27"
- board text removed: "Bypass R28"
- board text removed: "D1"
- board text removed: "HALL_SW_0"
- board text removed: "HALL_SW_1"
- board text removed: "I2C Address (All pins Low Default)"
- board text removed: "LED_1_2"
- board text removed: "MS1"
- board text removed: "MS2"
- board text removed: "Pins"
- board text removed: "Setting"
