File: electronics/KiCad/1_Distribution_Board/1_Distribution_Board.kicad_sch (KiCad schematic)
At the start: 12 parts, among them Q1 DMG2305UX, U1 KH-2.54FH-1X20P-H8.5, U2 KH-2.54FH-1X20P-H8.5

Commit message: Distribution board v1.4.1: effreek's revision, REV label, JLC rotation offsets restored (#1169)
effreek's pull-up/pull-down cleanup and test serial-servo circuit (J11/J14/J15), REV 1.4.1 on the board, the 33 JLC rotation offsets restored, test points out of the position file, and the V1.4.1 Gerber zip. Supersedes #1042.

Co-authored-by: effreek <115494910+effreek@users.noreply.github.com>
Co-Authored-By: Claude Opus 5.5 <noreply@anthropic.com>
Parts:
- added R21, R22, R27, R28, R61, R62, R63, R64, R67, R68: 10kΩ, PCM_JLCPCB:R_0603, symbol PCM_JLCPCB-Resistors:0603,10kΩ
- added R33: 2.2kΩ, PCM_JLCPCB:R_0603, symbol PCM_JLCPCB-Resistors:0603,2.2kΩ
- added R35: 100Ω, PCM_JLCPCB:R_0603, symbol PCM_JLCPCB-Resistors:0603,100Ω
- D1: LCSC (none) -> C223608; now fitted
Connections:
- net +3V3: now also R27.1, R33.2, R62.1, R63.1, R64.1
- net GND: now also R21.1, R22.1, R28.1, R61.1, R67.1, R68.1
- net GPIO2-GPIO_IN_HALL-SW_1 renamed GPIO2-GPIO_IN_OUT-SERIAL_SERVO
- net GPIO2-GPIO_IN_OUT-SERIAL_SERVO: now also R35.2
- net GPIO3-GPIO_IN_HALL-SW_0 renamed GPIO3-GPIO_IN-LIMIT_SWITCH
- new net SERIAL_SERVO: R33.1, R35.1
- new net Stepper Module/MS1: R21.2
- new net Stepper Module/MS2: R22.2
- new net Stepper Module1/MS1: R27.2
- new net Stepper Module1/MS2: R28.2
- new net Stepper Module2/MS1: R61.2
- new net Stepper Module2/MS2: R62.2
- new net Stepper Module3/MS1: R63.2
- new net Stepper Module3/MS2: R64.2
- new net Stepper Module4/MS1: R67.2
- new net Stepper Module4/MS2: R68.2
Other:
- sheet Hall_Switch_LED renamed Switch_LED
- sheet Power ports: added SERIAL_SERVO; removed none
- sheet Stepper Module ports: added MS1, MS2; removed none
- sheet Stepper Module1 ports: added MS1, MS2; removed none
- sheet Stepper Module2 ports: added MS1, MS2; removed none
- sheet Stepper Module3 ports: added MS1, MS2; removed none
- sheet Stepper Module4 ports: added MS1, MS2; removed none
- sheet Switch_LED ports: added none; removed HALL_SW_1
- note added: "Pull-Ups I2C lines for PCA9685"
- note added: "Pulled High. Servo's drive it low. Need to check signal on long run."
- note added: "Stepper UART addresses: MS1 = AD0, MS2 = AD1 (TMC2209 datasheet 4.1) UART0: A2 = 0, A3 = 1, A4 = 2, A5 = 3 UART1: A6 = 0 Must match TMC_UART_ADDRESSES in the firmware"
- note added: "TMC2209 Datasheet REV1.09 Pg. 20"
- note removed: "Pull-Ups for I2C lines for PCA9685"
- moved on the sheet: R1, R2, R3, R4, R5, S1
