File: electronics/KiCad/1_Distribution_Board/Stepper_Module.kicad_sch (KiCad schematic)
At the start: 14 parts, among them J21 Jumper Pins, J22 Jumper Pins, J23 JST PH, J24 Generic 2.54mm, P1 Header-Female-2.54_1x8, P2 Header-Female-2.54_1x2, P3 Header-Female-2.54_1x8

Commit message: Distribution board v1.4.1: effreek's revision, REV label, JLC rotation offsets restored (#1169)
effreek's pull-up/pull-down cleanup and test serial-servo circuit (J11/J14/J15), REV 1.4.1 on the board, the 33 JLC rotation offsets restored, test points out of the position file, and the V1.4.1 Gerber zip. Supersedes #1042.

Co-authored-by: effreek <115494910+effreek@users.noreply.github.com>
Co-Authored-By: Claude Opus 5.5 <noreply@anthropic.com>
Parts:
- removed J21, J22: Jumper Pins, Connector_PinHeader_2.54mm:PinHeader_1x03_P2.54mm_Vertical, symbol Connector_Generic:Conn_01x03
- removed R61, R62, R63, R64: 10kΩ, PCM_JLCPCB:R_0603, symbol PCM_JLCPCB-Resistors:0603,10kΩ
Connections:
- no-connect marks 3 -> 4
Other:
- note added: "1k from RX to TX on MCU necessary for single wire UART"
- note added: "UART address, set on root sheet"
- note removed: "10k from RX to TX on MCU necessary for single wire UART"
- note removed: "Jumper Pins allow for configuration High or Low on MS1 and MS2 by simply adding a jumper across pins 1-2 or 2-3"
- note removed: "MS1 MS2 Steps Interpolation GND GND 8 Yes to 256 VIO GND 2 Yes to 256 GND VIO 4 Yes to 256 VIO VIO 16 Yes to 256"
- note removed: "Micro Step Setting"
- note removed: "Requires 2 Jumpers JLCPCB # C5305"
- note removed: "See Micro Step Setting"
